Commit message: failed in change parameter

File: src/car_model/urdf/smart_copy.xacro (robot description, xacro)
@@ -62,6 +62,6 @@
       <origin xyz="0.05 0 ${base_collision_height}" rpy="0 0 ${PI/2}"/>
       <geometry>
-        <!-- <mesh filename="package://car_model/meshes/vehicle_body.dae"/> -->
-        <box size="${base_length} ${base_width} ${base_height}"/>
+        <mesh filename="package://car_model/meshes/vehicle_body.dae"/>
+        <!-- <box size="${base_length} ${base_width} ${base_height}"/> -->
       </geometry>
     </visual>
@@ -102,6 +102,6 @@
       <origin xyz="0 0 0" rpy="0 0 -${PI/2}"/>
       <geometry>
-        <!-- <mesh filename="package://car_model/meshes/wheel.dae"/> -->
-        <cylinder length="${rear_tyre_length}" radius="${rear_tyre_r}"/>
+        <mesh filename="package://car_model/meshes/wheel.dae"/>
+        <!-- <cylinder length="${rear_tyre_length}" radius="${rear_tyre_r}"/> -->
       </geometry>
     </visual>
@@ -135,5 +135,5 @@
       <origin xyz="0 0 0" rpy="0 0 ${PI/2}"/>
       <geometry>
-        <!-- <mesh filename="package://car_model/meshes/wheel.dae"/> -->
+        <mesh filename="package://car_model/meshes/wheel.dae"/>
         <cylinder length="${rear_tyre_length}" radius="${rear_tyre_r}"/>
       </geometry>
@@ -193,7 +193,6 @@
       <origin xyz="0 0 0" rpy="0 0 -${PI/2}"/>
       <geometry>
-        <!-- <mesh filename="package://car_model/meshes/wheel.dae"/> -->
+        <mesh filename="package://car_model/meshes/wheel.dae"/>
         <cylinder length="${front_tyre_length}" radius="${front_tyre_r}"/>
-          <!-- <cylinder length="${front_tyre_length}" radius="${front_tyre_r}"/> -->
       </geometry>
     </visual>
@@ -252,6 +251,6 @@
       <origin xyz="0 0 0" rpy="0 0 ${PI/2}"/>
       <geometry>
-        <!-- <mesh filename="package://car_model/meshes/wheel.dae"/> -->
-        <cylinder length="${front_tyre_length}" radius="${front_tyre_r}"/>
+        <mesh filename="package://car_model/meshes/wheel.dae"/>
+        <!-- <cylinder length="${front_tyre_length}" radius="${front_tyre_r}"/> -->
       </geometry>
     </visual>

File: src/car_model/urdf/smart_nomesh.xacro (robot description, xacro)
@@ -3,21 +3,7 @@
   <xacro:property name="PI" value="3.1415926835897931"/>
   <!-- base -->
-  <!-- <xacro:property name="base_length" value="2.695"/>
-  <xacro:property name="base_width" value="0.68"/>
-  <xacro:property name="base_height" value="1.370"/>
-  <xacro:property name="base_collision_height" value="0.875"/>
-  <xacro:property name="base_mass" value="956"/>
-  <xacro:property name="base_mass_ixx" value="343"/>
-  <xacro:property name="base_mass_iyy" value="728"/>
-  <xacro:property name="base_mass_izz" value="772"/> -->
-          <!-- VEHICLE.WIDTH = 0.19;
-        VEHICLE.LENGTH = 0.22;
-        VEHICLE.LF = 0.05;
-        VEHICLE.LB = 0.03;
-        VEHICLE.WHEEL_WIDTH = 0.018;
-        VEHICLE.WHEEL_LENGTH = 0.065;  -->
   <xacro:property name="base_length" value="0.22"/>
   <xacro:property name="base_width" value="0.19"/>
-  <xacro:property name="base_height" value="1.370"/>
+  <xacro:property name="base_height" value="0.1370"/>
   <xacro:property name="base_collision_height" value="0.875"/>
   <xacro:property name="base_mass" value="956"/>
@@ -60,7 +46,6 @@
     </collision>
     <visual>
-      <origin xyz="0.05 0 ${base_collision_height}" rpy="0 0 ${PI/2}"/>
-      <geometry>
-        <!-- <mesh filename="package://car_model/meshes/vehicle_body.dae"/> -->
+      <origin xyz="0 0 ${base_collision_height}" rpy="0 0 0"/>
+      <geometry>
         <box size="${base_length} ${base_width} ${base_height}"/>
       </geometry>
@@ -100,7 +85,6 @@
     </collision>
     <visual>
-      <origin xyz="0 0 0" rpy="0 0 -${PI/2}"/>
-      <geometry>
-        <!-- <mesh filename="package://car_model/meshes/wheel.dae"/> -->
+      <origin xyz="0 0 0" rpy="${PI/2} 0 0"/>
+      <geometry>
         <cylinder length="${rear_tyre_length}" radius="${rear_tyre_r}"/>
       </geometry>
@@ -133,7 +117,6 @@
     </collision>
     <visual>
-      <origin xyz="0 0 0" rpy="0 0 ${PI/2}"/>
-      <geometry>
-        <!-- <mesh filename="package://car_model/meshes/wheel.dae"/> -->
+      <origin xyz="0 0 0" rpy="${PI/2} 0 0"/>
+      <geometry>
         <cylinder length="${rear_tyre_length}" radius="${rear_tyre_r}"/>
       </geometry>
@@ -191,9 +174,7 @@
     </collision>
     <visual>
-      <origin xyz="0 0 0" rpy="0 0 -${PI/2}"/>
-      <geometry>
-        <!-- <mesh filename="package://car_model/meshes/wheel.dae"/> -->
+      <origin xyz="0 0 0" rpy="${PI/2} 0 0"/>
+      <geometry>
         <cylinder length="${front_tyre_length}" radius="${front_tyre_r}"/>
-          <!-- <cylinder length="${front_tyre_length}" radius="${front_tyre_r}"/> -->
       </geometry>
     </visual>
@@ -250,7 +231,6 @@
     </collision>
     <visual>
-      <origin xyz="0 0 0" rpy="0 0 ${PI/2}"/>
-      <geometry>
-        <!-- <mesh filename="package://car_model/meshes/wheel.dae"/> -->
+      <origin xyz="0 0 0" rpy="${PI/2} 0 0"/>
+      <geometry>
         <cylinder length="${front_tyre_length}" radius="${front_tyre_r}"/>
       </geometry>
